Commit message: renamed

File: yozakura_display/robot/arm.xacro (robot description, xacro)
@@ -1,8 +1,8 @@
 <?xml version="1.0"?>
-<robot name="newrobo" xmlns:xacro="http://www.ros.org/wiki/xacro">
+<robot name="yozakura" xmlns:xacro="http://www.ros.org/wiki/xacro">
 	<xacro:include filename="$(find xacro)/define.xacro" />
-	<xacro:include filename="$(find shinobi_newrobo_display)/robot/config.xacro" />
-	<xacro:include filename="$(find shinobi_newrobo_display)/robot/flipper_macro.xacro" />
-	<xacro:include filename="$(find shinobi_newrobo_display)/robot/starWheel_macro.xacro" />
+	<xacro:include filename="$(find yozakura_display)/robot/config.xacro" />
+	<xacro:include filename="$(find yozakura_display)/robot/flipper_macro.xacro" />
+	<xacro:include filename="$(find yozakura_display)/robot/starWheel_macro.xacro" />
 	<link name="arm_base">
 		<visual>

File: yozakura_display/robot/armjack_left_macro.xacro (robot description, xacro)
@@ -1,8 +1,26 @@
 <?xml version="1.0"?>
 <robot xmlns:xacro="http://www.ros.org/wiki/xacro">
-	<xacro:include filename="$(find shinobi_newrobo_display)/robot/config.xacro" />
-	<xacro:macro 	name="armjack_right"
+	<xacro:include filename="$(find yozakura_display)/robot/config.xacro" />
+	<xacro:macro 	name="armjack_left"
 								params="parent suffix">
-  <joint name="${joint_armLinear_right_A}_${suffix}" type="revolute">
+  <joint name="${joint_armLinear_left_A}_${suffix}" type="revolute">
+    <axis xyz="0 0 1"/>
+    <limit 	lower="${DEG2RAD*armYawAngle_min}" effort="1000.0"
+						upper="${DEG2RAD*armYawAngle_max}" velocity="0.5"/>
+    <origin rpy="0 0 0"
+						xyz="0 ${-armLinear_frame_length} 0"/>
+    <parent link="${parent}"/>
+    <child link="${arm_linear_frame_left_A}_${suffix}"/>
+  </joint>
+	<link name="${arm_linear_frame_left_A}_${suffix}">
+		<visual>
+			<origin rpy="0 0 0"
+							xyz="0 ${armLinear_frame_length/2.0} 0"/>
+			<geometry>
+				<mesh filename="${robotPackagePath}/${modelDataResourseFolder}/arm_linear_frame.stl"/>
+			</geometry>
+		</visual>
+	</link>
+  <joint name="${joint_armLinear_left_B}_${suffix}" type="revolute">
     <axis xyz="0 0 1"/>
     <limit 	lower="${DEG2RAD*armYawAngle_min}" effort="1000.0"
@@ -10,8 +28,8 @@
     <origin rpy="0 0 0"
 						xyz="0 ${armLinear_frame_length} 0"/>
-    <parent link="${parent}"/>
-    <child link="${arm_linear_frame_right_A}_${suffix}"/>
+    <parent link="${arm_linear_frame_left_A}_${suffix}"/>
+    <child link="${arm_linear_frame_left_B}_${suffix}"/>
   </joint>
-	<link name="${arm_linear_frame_right_A}_${suffix}">
+	<link name="${arm_linear_frame_left_B}_${suffix}">
 		<visual>
 			<origin rpy="0 0 0"
@@ -22,22 +40,4 @@
 		</visual>
 	</link>
-  <joint name="${joint_armLinear_right_B}_${suffix}" type="revolute">
-    <axis xyz="0 0 1"/>
-    <limit 	lower="${DEG2RAD*armYawAngle_min}" effort="1000.0"
-						upper="${DEG2RAD*armYawAngle_max}" velocity="0.5"/>
-    <origin rpy="0 0 0"
-						xyz="0 ${-armLinear_frame_length} 0"/>
-    <parent link="${arm_linear_frame_right_A}_${suffix}"/>
-    <child link="${arm_linear_frame_right_B}_${suffix}"/>
-  </joint>
-	<link name="${arm_linear_frame_right_B}_${suffix}">
-		<visual>
-			<origin rpy="0 0 0"
-							xyz="0 ${armLinear_frame_length/2.0} 0"/>
-			<geometry>
-				<mesh filename="${robotPackagePath}/${modelDataResourseFolder}/arm_linear_frame.stl"/>
-			</geometry>
-		</visual>
-	</link>
 	</xacro:macro>
 </robot>

File: yozakura_display/robot/armjack_right_macro.xacro (robot description, xacro)
@@ -1,8 +1,26 @@
 <?xml version="1.0"?>
 <robot xmlns:xacro="http://www.ros.org/wiki/xacro">
-	<xacro:include filename="$(find shinobi_newrobo_display)/robot/config.xacro" />
-	<xacro:macro 	name="armjack_left"
+	<xacro:include filename="$(find yozakura_display)/robot/config.xacro" />
+	<xacro:macro 	name="armjack_right"
 								params="parent suffix">
-  <joint name="${joint_armLinear_left_A}_${suffix}" type="revolute">
+  <joint name="${joint_armLinear_right_A}_${suffix}" type="revolute">
+    <axis xyz="0 0 1"/>
+    <limit 	lower="${DEG2RAD*armYawAngle_min}" effort="1000.0"
+						upper="${DEG2RAD*armYawAngle_max}" velocity="0.5"/>
+    <origin rpy="0 0 0"
+						xyz="0 ${armLinear_frame_length} 0"/>
+    <parent link="${parent}"/>
+    <child link="${arm_linear_frame_right_A}_${suffix}"/>
+  </joint>
+	<link name="${arm_linear_frame_right_A}_${suffix}">
+		<visual>
+			<origin rpy="0 0 0"
+							xyz="0 ${-armLinear_frame_length/2.0} 0"/>
+			<geometry>
+				<mesh filename="${robotPackagePath}/${modelDataResourseFolder}/arm_linear_frame.stl"/>
+			</geometry>
+		</visual>
+	</link>
+  <joint name="${joint_armLinear_right_B}_${suffix}" type="revolute">
     <axis xyz="0 0 1"/>
     <limit 	lower="${DEG2RAD*armYawAngle_min}" effort="1000.0"
@@ -10,8 +28,8 @@
     <origin rpy="0 0 0"
 						xyz="0 ${-armLinear_frame_length} 0"/>
-    <parent link="${parent}"/>
-    <child link="${arm_linear_frame_left_A}_${suffix}"/>
+    <parent link="${arm_linear_frame_right_A}_${suffix}"/>
+    <child link="${arm_linear_frame_right_B}_${suffix}"/>
   </joint>
-	<link name="${arm_linear_frame_left_A}_${suffix}">
+	<link name="${arm_linear_frame_right_B}_${suffix}">
 		<visual>
 			<origin rpy="0 0 0"
@@ -22,22 +40,4 @@
 		</visual>
 	</link>
-  <joint name="${joint_armLinear_left_B}_${suffix}" type="revolute">
-    <axis xyz="0 0 1"/>
-    <limit 	lower="${DEG2RAD*armYawAngle_min}" effort="1000.0"
-						upper="${DEG2RAD*armYawAngle_max}" velocity="0.5"/>
-    <origin rpy="0 0 0"
-						xyz="0 ${armLinear_frame_length} 0"/>
-    <parent link="${arm_linear_frame_left_A}_${suffix}"/>
-    <child link="${arm_linear_frame_left_B}_${suffix}"/>
-  </joint>
-	<link name="${arm_linear_frame_left_B}_${suffix}">
-		<visual>
-			<origin rpy="0 0 0"
-							xyz="0 ${-armLinear_frame_length/2.0} 0"/>
-			<geometry>
-				<mesh filename="${robotPackagePath}/${modelDataResourseFolder}/arm_linear_frame.stl"/>
-			</geometry>
-		</visual>
-	</link>
 	</xacro:macro>
 </robot>

File: yozakura_display/robot/config.xacro (robot description, xacro)
@@ -1,5 +1,5 @@
 <?xml version="1.0"?>
 <robot>
-	<property name="robotPackagePath" value="package://shinobi_newrobo_display/robot"/>
+	<property name="robotPackagePath" value="package://yozakura_display/robot"/>
 	<property name="modelDataResourseFolder" value="newRobotStls"/>
 	<property name="bodyFront_depth" 	value="0.262" />

File: yozakura_display/robot/flipper_macro.xacro (robot description, xacro)
@@ -1,5 +1,5 @@
 <?xml version="1.0"?>
 <robot xmlns:xacro="http://www.ros.org/wiki/xacro">
-	<xacro:include filename="$(find shinobi_newrobo_display)/robot/config.xacro" />
+	<xacro:include filename="$(find yozakura_display)/robot/config.xacro" />
 	<xacro:macro 	name="combine_lr_flippers"
 								params="left_joint_name right_joint_name parent flipper_tread suffix *origin">

File: yozakura_display/robot/starWheel_macro.xacro (robot description, xacro)
@@ -1,5 +1,5 @@
 <?xml version="1.0"?>
 <robot xmlns:xacro="http://www.ros.org/wiki/xacro">
-	<xacro:include filename="$(find shinobi_newrobo_display)/robot/config.xacro" />
+	<xacro:include filename="$(find yozakura_display)/robot/config.xacro" />
 	<xacro:macro 	name="combine_lr_wheels"
 								params="joint_name parent suffix wheel_tread *origin">

File: yozakura_display/robot/test.urdf.xacro (robot description, xacro)
@@ -1,8 +1,8 @@
 <?xml version="1.0"?>
-<robot name="newrobo" xmlns:xacro="http://www.ros.org/wiki/xacro">
+<robot name="yozakura" xmlns:xacro="http://www.ros.org/wiki/xacro">
 	<xacro:include filename="$(find xacro)/define.xacro" />
-	<xacro:include filename="$(find shinobi_newrobo_display)/robot/config.xacro" />
-	<xacro:include filename="$(find shinobi_newrobo_display)/robot/armjack_left_macro.xacro" />
-	<xacro:include filename="$(find shinobi_newrobo_display)/robot/armjack_right_macro.xacro" />
+	<xacro:include filename="$(find yozakura_display)/robot/config.xacro" />
+	<xacro:include filename="$(find yozakura_display)/robot/armjack_left_macro.xacro" />
+	<xacro:include filename="$(find yozakura_display)/robot/armjack_right_macro.xacro" />
 	<link name="arm_linear_frame_base">
 			<origin rpy="0 0 0" xyz="0 0 0"/>

File: yozakura_display/robot/yozakura.urdf.xacro (robot description, xacro)
@@ -1,10 +1,10 @@
 <?xml version="1.0"?>
-<robot name="newrobo" xmlns:xacro="http://www.ros.org/wiki/xacro">
-    <xacro:include filename="$(find shinobi_newrobo_display)/robot/define.xacro"/>
-    <xacro:include filename="$(find shinobi_newrobo_display)/robot/config.xacro"/>
-    <xacro:include filename="$(find shinobi_newrobo_display)/robot/flipper_macro.xacro"/>
-    <xacro:include filename="$(find shinobi_newrobo_display)/robot/starWheel_macro.xacro"/>
-    <xacro:include filename="$(find shinobi_newrobo_display)/robot/armjack_left_macro.xacro"/>
-    <xacro:include filename="$(find shinobi_newrobo_display)/robot/armjack_right_macro.xacro"/>
+<robot name="yozakura" xmlns:xacro="http://www.ros.org/wiki/xacro">
+    <xacro:include filename="$(find yozakura_display)/robot/define.xacro"/>
+    <xacro:include filename="$(find yozakura_display)/robot/config.xacro"/>
+    <xacro:include filename="$(find yozakura_display)/robot/flipper_macro.xacro"/>
+    <xacro:include filename="$(find yozakura_display)/robot/starWheel_macro.xacro"/>
+    <xacro:include filename="$(find yozakura_display)/robot/armjack_left_macro.xacro"/>
+    <xacro:include filename="$(find yozakura_display)/robot/armjack_right_macro.xacro"/>
     <!-- BODY -->
     <link name="virtualLink_world">

File: yozakura_display/robot/yozakura_arm.urdf.xacro (robot description, xacro)
@@ -1,8 +1,8 @@
 <?xml version="1.0"?>
-<robot name="newrobo" xmlns:xacro="http://www.ros.org/wiki/xacro">
+<robot name="yozakura" xmlns:xacro="http://www.ros.org/wiki/xacro">
 	<xacro:include filename="$(find xacro)/define.xacro" />
-	<xacro:include filename="$(find shinobi_newrobo_display)/robot/config.xacro" />
-	<xacro:include filename="$(find shinobi_newrobo_display)/robot/armjack_left_macro.xacro" />
-	<xacro:include filename="$(find shinobi_newrobo_display)/robot/armjack_right_macro.xacro" />
+	<xacro:include filename="$(find yozakura_display)/robot/config.xacro" />
+	<xacro:include filename="$(find yozakura_display)/robot/armjack_left_macro.xacro" />
+	<xacro:include filename="$(find yozakura_display)/robot/armjack_right_macro.xacro" />
 	<!-- ARM BASE -->
 	<link name="arm_base">

File: yozakura_display/robot/yozakura_body.urdf.xacro (robot description, xacro)
@@ -1,10 +1,10 @@
 <?xml version="1.0"?>
-<robot name="newrobo" xmlns:xacro="http://www.ros.org/wiki/xacro">
+<robot name="yozakura" xmlns:xacro="http://www.ros.org/wiki/xacro">
 	<xacro:include filename="$(find xacro)/define.xacro" />
-	<xacro:include filename="$(find shinobi_newrobo_display)/robot/config.xacro" />
-	<xacro:include filename="$(find shinobi_newrobo_display)/robot/flipper_macro.xacro" />
-	<xacro:include filename="$(find shinobi_newrobo_display)/robot/starWheel_macro.xacro" />
-	<xacro:include filename="$(find shinobi_newrobo_display)/robot/armjack_left_macro.xacro" />
-	<xacro:include filename="$(find shinobi_newrobo_display)/robot/armjack_right_macro.xacro" />
+	<xacro:include filename="$(find yozakura_display)/robot/config.xacro" />
+	<xacro:include filename="$(find yozakura_display)/robot/flipper_macro.xacro" />
+	<xacro:include filename="$(find yozakura_display)/robot/starWheel_macro.xacro" />
+	<xacro:include filename="$(find yozakura_display)/robot/armjack_left_macro.xacro" />
+	<xacro:include filename="$(find yozakura_display)/robot/armjack_right_macro.xacro" />
 	<!-- BODY -->
 	<link name="body_front">
