Commit message: rename and remove unnecessary files

File: yozakura_display/robot/arm.xacro (robot description, xacro)
@@ -1,54 +1,46 @@
 <?xml version="1.0"?>
 <robot name="yozakura" xmlns:xacro="http://www.ros.org/wiki/xacro">
-	<xacro:include filename="$(find xacro)/define.xacro" />
-	<xacro:include filename="$(find yozakura_display)/robot/config.xacro" />
-	<xacro:include filename="$(find yozakura_display)/robot/flipper_macro.xacro" />
-	<xacro:include filename="$(find yozakura_display)/robot/starWheel_macro.xacro" />
-	<link name="arm_base">
-		<visual>
-			<origin rpy="0 0 0"
-							xyz="0 0 0"/>
-			<geometry>
-				<mesh filename="${robotPackagePath}/${modelDataResourseFolder}/arm_base.stl"/>
-			</geometry>
-		</visual>
-	</link>
-  <joint name="joint_arm_yaw" type="revolute">
-    <axis xyz="0 0 1"/>
-    <limit 	lower="${DEG2RAD*armYawAngle_min}" effort="1000.0"
-						upper="${DEG2RAD*armYawAngle_max}" velocity="0.5"/>
-    <origin rpy="0 0 0"
-						xyz="0 0 ${armYawStage_fromBodyTop}"/>
-    <parent link="arm_base"/>
-    <child link="arm_yaw"/>
-  </joint>
-	<link name="arm_yaw">
-		<visual>
-			<origin rpy="0 0 0"
-							xyz="0 0 0"/>
-			<geometry>
-				<mesh filename="${robotPackagePath}/${modelDataResourseFolder}/arm_yaw.stl"/>
-			</geometry>
-		</visual>
-	</link>
-  <joint name="joint_arm_pitch" type="revolute">
-    <axis xyz="0 1 0"/>
-    <limit 	lower="${DEG2RAD*armPitchAngle_min}" effort="1000.0"
-						upper="${DEG2RAD*armPitchAngle_max}" velocity="0.5"/>
-    <origin rpy="0 0 0"
-						xyz="${-armPitchAxis_fromYawAxis} 0 ${armPitchAxis_fromYawStage}"/>
-    <parent link="arm_yaw"/>
-    <child link="arm_pitch"/>
-  </joint>
-	<link name="arm_pitch">
-		<visual>
-			<origin rpy="0 0 0"
-							xyz="${-armLinearAxis_fromPitchAxis}
-									0
-									${-armPitchAxis_fromYawStage + armLinearAxis_fromYawStage}"/>
-			<geometry>
-				<mesh filename="${robotPackagePath}/${modelDataResourseFolder}/arm_pitch.stl"/>
-			</geometry>
-		</visual>
-	</link>
+    <xacro:include filename="$(find xacro)/define.xacro"/>
+    <xacro:include filename="$(find yozakura_display)/robot/config.xacro"/>
+    <xacro:include filename="$(find yozakura_display)/robot/flipper_macro.xacro"/>
+    <xacro:include filename="$(find yozakura_display)/robot/wheel_macro.xacro"/>
+    <link name="virtual_arm_base">
+        <origin rpy="0 0 0" xyz="0 0 0"/>
+    </link>
+    <joint name="joint_arm_yaw" type="revolute">
+        <axis xyz="0 0 1"/>
+        <limit lower="${DEG2RAD*armYawAngle_min}" effort="1000.0"
+               upper="${DEG2RAD*armYawAngle_max}" velocity="0.5"/>
+        <origin rpy="0 0 0"
+                xyz="0 0 ${armYawStage_fromBodyTop}"/>
+        <parent link="virtual_arm_base"/>
+        <child link="arm_yaw"/>
+    </joint>
+    <link name="arm_yaw">
+        <visual>
+            <origin rpy="0 0 0"
+                    xyz="0 0 0"/>
+            <geometry>
+                <mesh filename="${robotPackagePath}/${modelDataResourseFolder}/arm_yaw.dae"/>
+            </geometry>
+        </visual>
+    </link>
+    <joint name="joint_arm_pitch" type="revolute">
+        <axis xyz="0 1 0"/>
+        <limit lower="${DEG2RAD*armPitchAngle_min}" effort="1000.0"
+               upper="${DEG2RAD*armPitchAngle_max}" velocity="0.5"/>
+        <origin rpy="0 0 0"
+                xyz="${-armPitchAxis_fromYawAxis} 0 ${armPitchAxis_fromYawStage}"/>
+        <parent link="arm_yaw"/>
+        <child link="arm_pitch"/>
+    </joint>
+    <link name="arm_pitch">
+        <visual>
+            <origin rpy="0 0 0"
+                    xyz="${-armLinearAxis_fromPitchAxis} 0 ${-armPitchAxis_fromYawStage + armLinearAxis_fromYawStage}"/>
+            <geometry>
+                <mesh filename="${robotPackagePath}/${modelDataResourseFolder}/arm_pitch.dae"/>
+            </geometry>
+        </visual>
+    </link>
 </robot>

File: yozakura_display/robot/armjack_left_macro.xacro (robot description, xacro)
@@ -1,43 +1,42 @@
 <?xml version="1.0"?>
 <robot xmlns:xacro="http://www.ros.org/wiki/xacro">
-	<xacro:include filename="$(find yozakura_display)/robot/config.xacro" />
-	<xacro:macro 	name="armjack_left"
-								params="parent suffix">
-  <joint name="${joint_armLinear_left_A}_${suffix}" type="revolute">
-    <axis xyz="0 0 1"/>
-    <limit 	lower="${DEG2RAD*armYawAngle_min}" effort="1000.0"
-						upper="${DEG2RAD*armYawAngle_max}" velocity="0.5"/>
-    <origin rpy="0 0 0"
-						xyz="0 ${-armLinear_frame_length} 0"/>
-    <parent link="${parent}"/>
-    <child link="${arm_linear_frame_left_A}_${suffix}"/>
-  </joint>
-	<link name="${arm_linear_frame_left_A}_${suffix}">
-		<visual>
-			<origin rpy="0 0 0"
-							xyz="0 ${armLinear_frame_length/2.0} 0"/>
-			<geometry>
-				<mesh filename="${robotPackagePath}/${modelDataResourseFolder}/arm_linear_frame.stl"/>
-			</geometry>
-		</visual>
-	</link>
-  <joint name="${joint_armLinear_left_B}_${suffix}" type="revolute">
-    <axis xyz="0 0 1"/>
-    <limit 	lower="${DEG2RAD*armYawAngle_min}" effort="1000.0"
-						upper="${DEG2RAD*armYawAngle_max}" velocity="0.5"/>
-    <origin rpy="0 0 0"
-						xyz="0 ${armLinear_frame_length} 0"/>
-    <parent link="${arm_linear_frame_left_A}_${suffix}"/>
-    <child link="${arm_linear_frame_left_B}_${suffix}"/>
-  </joint>
-	<link name="${arm_linear_frame_left_B}_${suffix}">
-		<visual>
-			<origin rpy="0 0 0"
-							xyz="0 ${-armLinear_frame_length/2.0} 0"/>
-			<geometry>
-				<mesh filename="${robotPackagePath}/${modelDataResourseFolder}/arm_linear_frame.stl"/>
-			</geometry>
-		</visual>
-	</link>
-	</xacro:macro>
+    <xacro:include filename="$(find yozakura_display)/robot/config.xacro"/>
+    <xacro:macro name="armjack_left" params="parent suffix">
+        <joint name="${joint_armLinear_left_A}_${suffix}" type="revolute">
+            <axis xyz="0 0 1"/>
+            <limit lower="${DEG2RAD*armYawAngle_min}" effort="1000.0"
+                   upper="${DEG2RAD*armYawAngle_max}" velocity="0.5"/>
+            <origin rpy="0 0 0"
+                    xyz="0 ${-armLinear_frame_length} 0"/>
+            <parent link="${parent}"/>
+            <child link="${arm_linear_frame_left_A}_${suffix}"/>
+        </joint>
+        <link name="${arm_linear_frame_left_A}_${suffix}">
+            <visual>
+                <origin rpy="0 0 0"
+                        xyz="0 ${armLinear_frame_length/2.0} 0"/>
+                <geometry>
+                    <mesh filename="${robotPackagePath}/${modelDataResourseFolder}/arm_linear_frame.stl"/>
+                </geometry>
+            </visual>
+        </link>
+        <joint name="${joint_armLinear_left_B}_${suffix}" type="revolute">
+            <axis xyz="0 0 1"/>
+            <limit lower="${DEG2RAD*armYawAngle_min}" effort="1000.0"
+                   upper="${DEG2RAD*armYawAngle_max}" velocity="0.5"/>
+            <origin rpy="0 0 0"
+                    xyz="0 ${armLinear_frame_length} 0"/>
+            <parent link="${arm_linear_frame_left_A}_${suffix}"/>
+            <child link="${arm_linear_frame_left_B}_${suffix}"/>
+        </joint>
+        <link name="${arm_linear_frame_left_B}_${suffix}">
+            <visual>
+                <origin rpy="0 0 0"
+                        xyz="0 ${-armLinear_frame_length/2.0} 0"/>
+                <geometry>
+                    <mesh filename="${robotPackagePath}/${modelDataResourseFolder}/arm_linear_frame.stl"/>
+                </geometry>
+            </visual>
+        </link>
+    </xacro:macro>
 </robot>

File: yozakura_display/robot/config.xacro (robot description, xacro)
@@ -1,51 +1,54 @@
 <?xml version="1.0"?>
 <robot>
-	<property name="robotPackagePath" value="package://yozakura_display/robot"/>
-	<property name="modelDataResourseFolder" value="newRobotStls"/>
-	<property name="bodyFront_depth" 	value="0.262" />
-  <property name="bodyFront_height" value="0.072" />
-  <property name="bodyFront_width" 	value="0.262" />
-	<property name="bodyPitchAngle_max"	value=  "0" />
-	<property name="bodyPitchAngle_min"	value="-90" />
-	<property name="bodyLink_length" value="0.038" />
-  <property name="bodyBack_depth" 	value="0.112" />
-  <property name="bodyBack_height" 	value="0.072" />
-  <property name="bodyBack_width" 	value="0.340" />
-  <property name="starWheel_width" 	value="0.018" />
-  <property name="starWheel_radius" value="0.134" />
-  <property name="starWheelAxis_radius" value="0.134" />
-	<property name="frontwheelAxis_fromBodyCenter" value="0.070" />
-  <property name="backwheelAxis_fromBodyCenter" value="-0.100" />
-	<property name="frontwheel_tread" value="0.372"/> <!-- from outside to outside -->
-  <property name="backwheel_tread" value="0.386"/> <!-- from outside to outside -->
-  <property name="flipper_width" 		value="0.025" />
-  <property name="flipper_length" 	value="0.178" />
-  <property name="flipper_tread" 	value="0.320" /> <!-- from outside to outside -->
-  <property name="flipperBigPulley_radius" value="0.032" />
-  <property name="flipperAngle_max" value= "90" />
-  <property name="flipperAngle_min" value="-90" />
-  <property name="flipperAxis_fromBodyCenter" value="0.070" />
-  <property name="flipperOffset_fromBodySide" value="0.010" />
-	<property name="armYawAngle_max"	value= "90" />
-	<property name="armYawAngle_min"	value="-90" />
-	<property name="armPitchAngle_max"	value= "90" />
-	<property name="armPitchAngle_min"	value="-90" />
-  <property name="armBase_fromBodyCenter_X" value="0.040" />
-  <property name="armYawStage_fromBodyTop" value="0.020" />
-  <property name="armPitchAxis_fromYawAxis" value="0.045" />
-  <property name="armPitchAxis_fromYawStage" value="0.045" />
-  <property name="armLinearAxis_fromPitchAxis" value="0.010" />
-  <property name="armLinearAxis_fromYawStage" value="0.055" />
-	<property name="armLinearBase_ArmLinearAxis" value="0.025" />
-  <property name="armLinear_frame_length" value="0.200" />
-  <property name="arm_linear_frame_left_A" value="arm_linear_frame_left_A" />
-  <property name="arm_linear_frame_left_B" value="arm_linear_frame_left_B" />
-  <property name="joint_armLinear_left_A" value="joint_armLinear_left_A" />
-  <property name="joint_armLinear_left_B" value="joint_armLinear_left_B" />
-  <property name="joint_armLinear_left_C" value="joint_armLinear_left_C" />
-  <property name="arm_linear_frame_right_A" value="arm_linear_frame_right_A" />
-  <property name="arm_linear_frame_right_B" value="arm_linear_frame_right_B" />
-  <property name="joint_armLinear_right_A" value="joint_armLinear_right_A" />
-  <property name="joint_armLinear_right_B" value="joint_armLinear_right_B" />
-  <property name="joint_armLinear_right_C" value="joint_armLinear_right_C" />
+    <property name="robotPackagePath" value="package://yozakura_display/robot"/>
+    <property name="modelDataResourseFolder" value="daes"/>
+    <property name="bodyFront_depth" value="0.262"/>
+    <property name="bodyFront_height" value="0.072"/>
+    <property name="bodyFront_width" value="0.262"/>
+    <property name="bodyPitchAngle_max" value="0"/>
+    <property name="bodyPitchAngle_min" value="-90"/>
+    <property name="bodyLink_length" value="0.038"/>
+    <property name="bodyBack_depth" value="0.112"/>
+    <property name="bodyBack_height" value="0.072"/>
+    <property name="bodyBack_width" value="0.340"/>
+    <property name="starWheel_width" value="0.018"/>
+    <property name="starWheel_radius" value="0.134"/>
+    <property name="starWheelAxis_radius" value="0.134"/>
+    <property name="frontwheelAxis_fromBodyCenter" value="0.070"/>
+    <property name="backwheelAxis_fromBodyCenter" value="-0.100"/>
+    <property name="frontwheel_tread" value="0.372"/>
+    <!-- from outside to outside -->
+    <property name="backwheel_tread" value="0.386"/>
+    <!-- from outside to outside -->
+    <property name="flipper_width" value="0.025"/>
+    <property name="flipper_length" value="0.178"/>
+    <property name="flipper_tread" value="0.320"/>
+    <!-- from outside to outside -->
+    <property name="flipperBigPulley_radius" value="0.032"/>
+    <property name="flipperAngle_max" value="90"/>
+    <property name="flipperAngle_min" value="-90"/>
+    <property name="flipperAxis_fromBodyCenter" value="0.070"/>
+    <property name="flipperOffset_fromBodySide" value="0.010"/>
+    <property name="armYawAngle_max" value="90"/>
+    <property name="armYawAngle_min" value="-90"/>
+    <property name="armPitchAngle_max" value="90"/>
+    <property name="armPitchAngle_min" value="-90"/>
+    <property name="armBase_fromBodyCenter_X" value="0.040"/>
+    <property name="armYawStage_fromBodyTop" value="0.020"/>
+    <property name="armPitchAxis_fromYawAxis" value="0.045"/>
+    <property name="armPitchAxis_fromYawStage" value="0.045"/>
+    <property name="armLinearAxis_fromPitchAxis" value="0.010"/>
+    <property name="armLinearAxis_fromYawStage" value="0.055"/>
+    <property name="armLinearBase_ArmLinearAxis" value="0.025"/>
+    <property name="armLinear_frame_length" value="0.200"/>
+    <property name="arm_linear_frame_left_A" value="arm_linear_frame_left_A"/>
+    <property name="arm_linear_frame_left_B" value="arm_linear_frame_left_B"/>
+    <property name="joint_armLinear_left_A" value="joint_armLinear_left_A"/>
+    <property name="joint_armLinear_left_B" value="joint_armLinear_left_B"/>
+    <property name="joint_armLinear_left_C" value="joint_armLinear_left_C"/>
+    <property name="arm_linear_frame_right_A" value="arm_linear_frame_right_A"/>
+    <property name="arm_linear_frame_right_B" value="arm_linear_frame_right_B"/>
+    <property name="joint_armLinear_right_A" value="joint_armLinear_right_A"/>
+    <property name="joint_armLinear_right_B" value="joint_armLinear_right_B"/>
+    <property name="joint_armLinear_right_C" value="joint_armLinear_right_C"/>
 </robot>

File: yozakura_display/robot/yozakura.urdf.xacro (robot description, xacro)
@@ -4,5 +4,5 @@
     <xacro:include filename="$(find yozakura_display)/robot/config.xacro"/>
     <xacro:include filename="$(find yozakura_display)/robot/flipper_macro.xacro"/>
-    <xacro:include filename="$(find yozakura_display)/robot/starWheel_macro.xacro"/>
+    <xacro:include filename="$(find yozakura_display)/robot/wheel_macro.xacro"/>
     <xacro:include filename="$(find yozakura_display)/robot/armjack_left_macro.xacro"/>
     <xacro:include filename="$(find yozakura_display)/robot/armjack_right_macro.xacro"/>
@@ -33,5 +33,5 @@
                     xyz="0 0 0"/>
             <geometry>
-                <mesh filename="${robotPackagePath}/${modelDataResourseFolder}/body_front.stl"/>
+                <mesh filename="${robotPackagePath}/${modelDataResourseFolder}/body_front.dae"/>
             </geometry>
         </visual>
@@ -51,5 +51,5 @@
                     xyz="${-bodyLink_length/2.0} 0 ${bodyFront_height/2.0}"/>
             <geometry>
-                <mesh filename="${robotPackagePath}/${modelDataResourseFolder}/body_link.stl"/>
+                <mesh filename="${robotPackagePath}/${modelDataResourseFolder}/body_link.dae"/>
             </geometry>
         </visual>
@@ -67,5 +67,5 @@
                     xyz="${-bodyLink_length - bodyBack_depth/2.0} 0 ${bodyBack_height/2.0}"/>
             <geometry>
-                <mesh filename="${robotPackagePath}/${modelDataResourseFolder}/body_back.stl"/>
+                <mesh filename="${robotPackagePath}/${modelDataResourseFolder}/body_back.dae"/>
             </geometry>
         </visual>
@@ -94,13 +94,8 @@
         <origin rpy="0 0 0" xyz="${-armBase_fromBodyCenter_X} 0 ${bodyFront_height/2.0}"/>
         <parent link="body_front"/>
-        <child link="arm_base"/>
+        <child link="virtual_arm_base"/>
     </joint>
-    <link name="arm_base">
-        <visual>
-            <origin rpy="0 0 0" xyz="0 0 0"/>
-            <geometry>
-                <mesh filename="${robotPackagePath}/${modelDataResourseFolder}/arm_base.stl"/>
-            </geometry>
-        </visual>
+    <link name="virtual_arm_base">
+        <origin rpy="0 0 0" xyz="0 0 0"/>
     </link>
     <joint name="joint_arm_yaw" type="revolute">
@@ -110,5 +105,5 @@
         <origin rpy="0 0 0"
                 xyz="0 0 ${armYawStage_fromBodyTop}"/>
-        <parent link="arm_base"/>
+        <parent link="virtual_arm_base"/>
         <child link="arm_yaw"/>
     </joint>
@@ -118,5 +113,5 @@
                     xyz="0 0 0"/>
             <geometry>
-                <mesh filename="${robotPackagePath}/${modelDataResourseFolder}/arm_yaw.stl"/>
+                <mesh filename="${robotPackagePath}/${modelDataResourseFolder}/arm_yaw.dae"/>
             </geometry>
         </visual>
@@ -136,5 +131,5 @@
                     xyz="${-armLinearAxis_fromPitchAxis} 0	${-armPitchAxis_fromYawStage + armLinearAxis_fromYawStage}"/>
             <geometry>
-                <mesh filename="${robotPackagePath}/${modelDataResourseFolder}/arm_pitch.stl"/>
+                <mesh filename="${robotPackagePath}/${modelDataResourseFolder}/arm_pitch.dae"/>
             </geometry>
         </visual>
