Commit message: make sure that the colored urdf works

File: yozakura_display/robot/armjack_left_macro.xacro (robot description, xacro)
@@ -17,5 +17,5 @@
                         xyz="0 ${armLinear_frame_length/2.0} 0"/>
                 <geometry>
-                    <mesh filename="${robotPackagePath}/${modelDataResourseFolder}/arm_linear_frame.stl"/>
+                    <mesh filename="${robotPackagePath}/${modelDataResourseFolder}/arm_frame.dae"/>
                 </geometry>
             </visual>
@@ -35,5 +35,5 @@
                         xyz="0 ${-armLinear_frame_length/2.0} 0"/>
                 <geometry>
-                    <mesh filename="${robotPackagePath}/${modelDataResourseFolder}/arm_linear_frame.stl"/>
+                    <mesh filename="${robotPackagePath}/${modelDataResourseFolder}/arm_frame.dae"/>
                 </geometry>
             </visual>

File: yozakura_display/robot/armjack_right_macro.xacro (robot description, xacro)
@@ -18,5 +18,5 @@
 							xyz="0 ${-armLinear_frame_length/2.0} 0"/>
 			<geometry>
-				<mesh filename="${robotPackagePath}/${modelDataResourseFolder}/arm_linear_frame.stl"/>
+				<mesh filename="${robotPackagePath}/${modelDataResourseFolder}/arm_frame.dae"/>
 			</geometry>
 		</visual>
@@ -36,5 +36,5 @@
 							xyz="0 ${armLinear_frame_length/2.0} 0"/>
 			<geometry>
-				<mesh filename="${robotPackagePath}/${modelDataResourseFolder}/arm_linear_frame.stl"/>
+				<mesh filename="${robotPackagePath}/${modelDataResourseFolder}/arm_frame.dae"/>
 			</geometry>
 		</visual>

File: yozakura_display/robot/flipper_macro.xacro (robot description, xacro)
@@ -1,50 +1,50 @@
 <?xml version="1.0"?>
 <robot xmlns:xacro="http://www.ros.org/wiki/xacro">
-	<xacro:include filename="$(find yozakura_display)/robot/config.xacro" />
-	<xacro:macro 	name="combine_lr_flippers"
-								params="left_joint_name right_joint_name parent flipper_tread suffix *origin">
-	<!-- Axis -->
-		<joint name="fixedJoint_flipperAxis_${suffix}" type="fixed">
-			<insert_block name="origin" />
-  	  <parent link="${parent}" />
-  	  <child link="virtualLink_flipperAxis_${suffix}"/>
-  	</joint>
-		<link name="virtualLink_flipperAxis_${suffix}" />
-	<!-- left -->
-		<joint name="${left_joint_name}" type="revolute">
-  	  <axis xyz="0 1 0"/>
-			<origin rpy="0 0 0"
-							xyz="0 ${flipper_tread/2.0} 0" />
-    	<limit 	lower="${DEG2RAD*flipperAngle_min}" effort="1000.0"
-							upper="${DEG2RAD*flipperAngle_max}" velocity="0.5"/>
-  	  <parent link="virtualLink_flipperAxis_${suffix}"/>
-  	  <child link="flippper_left_${suffix}"/>
-  	</joint>
-		<link name="flippper_left_${suffix}">
-			<visual>
-				<origin rpy="0 0 0" xyz="0 0 0"/>
-				<geometry>
-					<mesh filename="${robotPackagePath}/${modelDataResourseFolder}/flipper_left.stl"/>
-				</geometry>
-			</visual>
-		</link>
-	<!-- right -->
-		<joint name="${right_joint_name}" type="revolute">
-  	  <axis xyz="0 1 0"/>
-			<origin rpy="0 0 0"
-							xyz="0 ${-flipper_tread/2.0} 0" />
-    	<limit 	lower="${DEG2RAD*flipperAngle_min}" effort="1000.0"
-							upper="${DEG2RAD*flipperAngle_max}" velocity="0.5"/>
-  	  <parent link="virtualLink_flipperAxis_${suffix}"/>
-  	  <child link="flipper_right_${suffix}"/>
-  	</joint>
-		<link name="flipper_right_${suffix}">
-			<visual>
-				<origin rpy="0 0 0" xyz="0 0 0"/>
-				<geometry>
-					<mesh filename="${robotPackagePath}/${modelDataResourseFolder}/flipper_right.stl"/>
-				</geometry>
-			</visual>
-		</link>
-	</xacro:macro>
+    <xacro:include filename="$(find yozakura_display)/robot/config.xacro"/>
+    <xacro:macro name="combine_lr_flippers"
+                 params="left_joint_name right_joint_name parent flipper_tread suffix *origin">
+        <!-- Axis -->
+        <joint name="fixedJoint_flipperAxis_${suffix}" type="fixed">
+            <insert_block name="origin"/>
+            <parent link="${parent}"/>
+            <child link="virtualLink_flipperAxis_${suffix}"/>
+        </joint>
+        <link name="virtualLink_flipperAxis_${suffix}"/>
+        <!-- left -->
+        <joint name="${left_joint_name}" type="revolute">
+            <axis xyz="0 1 0"/>
+            <origin rpy="0 0 0"
+                    xyz="0 ${flipper_tread/2.0} 0"/>
+            <limit lower="${DEG2RAD*flipperAngle_min}" effort="1000.0"
+                   upper="${DEG2RAD*flipperAngle_max}" velocity="0.5"/>
+            <parent link="virtualLink_flipperAxis_${suffix}"/>
+            <child link="flippper_left_${suffix}"/>
+        </joint>
+        <link name="flippper_left_${suffix}">
+            <visual>
+                <origin rpy="0 0 0" xyz="0 0 0"/>
+                <geometry>
+                    <mesh filename="${robotPackagePath}/${modelDataResourseFolder}/flipper_left.dae"/>
+                </geometry>
+            </visual>
+        </link>
+        <!-- right -->
+        <joint name="${right_joint_name}" type="revolute">
+            <axis xyz="0 1 0"/>
+            <origin rpy="0 0 0"
+                    xyz="0 ${-flipper_tread/2.0} 0"/>
+            <limit lower="${DEG2RAD*flipperAngle_min}" effort="1000.0"
+                   upper="${DEG2RAD*flipperAngle_max}" velocity="0.5"/>
+            <parent link="virtualLink_flipperAxis_${suffix}"/>
+            <child link="flipper_right_${suffix}"/>
+        </joint>
+        <link name="flipper_right_${suffix}">
+            <visual>
+                <origin rpy="0 0 0" xyz="0 0 0"/>
+                <geometry>
+                    <mesh filename="${robotPackagePath}/${modelDataResourseFolder}/flipper_right.dae"/>
+                </geometry>
+            </visual>
+        </link>
+    </xacro:macro>
 </robot>

File: yozakura_display/robot/wheel_macro.xacro (robot description, xacro)
@@ -1,45 +1,45 @@
 <?xml version="1.0"?>
 <robot xmlns:xacro="http://www.ros.org/wiki/xacro">
-	<xacro:include filename="$(find yozakura_display)/robot/config.xacro" />
-	<xacro:macro 	name="combine_lr_wheels"
-								params="joint_name parent suffix wheel_tread *origin">
-	<!-- Axis -->
-		<joint name="${joint_name}" type="continuous">
-  	  <axis xyz="0 1 0"/>
-			<insert_block name="origin" />
-  	  <parent link="${parent}"/>
-  	  <child link="virtual_starWheelAxisLink_${suffix}"/>
-  	</joint>
-		<link name="virtual_starWheelAxisLink_${suffix}" />
-	<!-- left -->
-		<joint name="fixedJoint_left_${suffix}" type="fixed">
-			<parent link="virtual_starWheelAxisLink_${suffix}"/>
-  	  <child  link="starWheel_left_${suffix}"/>
-  	  <origin xyz="0 ${wheel_tread/2.0} 0"/>
-		</joint>
-		<link name="starWheel_left_${suffix}">
-			<visual>
-				<origin rpy="0 0 0"
-								xyz="0 0 0"/>
-				<geometry>
-					<mesh filename="${robotPackagePath}/${modelDataResourseFolder}/wheel_left.stl"/>
-				</geometry>
-			</visual>
-		</link>
-	<!-- right -->
-		<joint name="fixedJoint_right_${suffix}" type="fixed">
-			<parent link="virtual_starWheelAxisLink_${suffix}"/>
-  	  <child  link="starWheel_right_${suffix}"/>
-  	  <origin xyz="0 ${-wheel_tread/2.0} 0"/>
-		</joint>
-		<link name="starWheel_right_${suffix}">
-			<visual>
-				<origin rpy="0 0 0"
-								xyz="0 0 0"/>
-				<geometry>
-					<mesh filename="${robotPackagePath}/${modelDataResourseFolder}/wheel_right.stl"/>
-				</geometry>
-			</visual>
-		</link>
-	</xacro:macro>
+    <xacro:include filename="$(find yozakura_display)/robot/config.xacro"/>
+    <xacro:macro name="combine_lr_wheels"
+                 params="joint_name parent suffix wheel_tread *origin">
+        <!-- Axis -->
+        <joint name="${joint_name}" type="continuous">
+            <axis xyz="0 1 0"/>
+            <insert_block name="origin"/>
+            <parent link="${parent}"/>
+            <child link="virtual_starWheelAxisLink_${suffix}"/>
+        </joint>
+        <link name="virtual_starWheelAxisLink_${suffix}"/>
+        <!-- left -->
+        <joint name="fixedJoint_left_${suffix}" type="fixed">
+            <parent link="virtual_starWheelAxisLink_${suffix}"/>
+            <child link="starWheel_left_${suffix}"/>
+            <origin xyz="0 ${wheel_tread/2.0} 0"/>
+        </joint>
+        <link name="starWheel_left_${suffix}">
+            <visual>
+                <origin rpy="0 0 0"
+                        xyz="0 0 0"/>
+                <geometry>
+                    <mesh filename="${robotPackagePath}/${modelDataResourseFolder}/wheel_left.dae"/>
+                </geometry>
+            </visual>
+        </link>
+        <!-- right -->
+        <joint name="fixedJoint_right_${suffix}" type="fixed">
+            <parent link="virtual_starWheelAxisLink_${suffix}"/>
+            <child link="starWheel_right_${suffix}"/>
+            <origin xyz="0 ${-wheel_tread/2.0} 0"/>
+        </joint>
+        <link name="starWheel_right_${suffix}">
+            <visual>
+                <origin rpy="0 0 0"
+                        xyz="0 0 0"/>
+                <geometry>
+                    <mesh filename="${robotPackagePath}/${modelDataResourseFolder}/wheel_right.dae"/>
+                </geometry>
+            </visual>
+        </link>
+    </xacro:macro>
 </robot>

File: yozakura_display/robot/yozakura.urdf.xacro (robot description, xacro)
@@ -3,92 +3,12 @@
     <xacro:include filename="$(find yozakura_display)/robot/define.xacro"/>
     <xacro:include filename="$(find yozakura_display)/robot/config.xacro"/>
-    <xacro:include filename="$(find yozakura_display)/robot/flipper_macro.xacro"/>
-    <xacro:include filename="$(find yozakura_display)/robot/wheel_macro.xacro"/>
-    <xacro:include filename="$(find yozakura_display)/robot/armjack_left_macro.xacro"/>
-    <xacro:include filename="$(find yozakura_display)/robot/armjack_right_macro.xacro"/>
+    <xacro:include filename="$(find yozakura_display)/robot/yozakura_arm.urdf.xacro"/>
+    <xacro:include filename="$(find yozakura_display)/robot/yozakura_body.urdf.xacro"/>
     <!-- BODY -->
-    <link name="virtualLink_world">
+    <link name="root">
         <origin rpy="0 0 0" xyz="0 0 0"/>
     </link>
-    <joint name="joint_body_front_pitch" type="continuous">
-        <axis xyz="0 1 0"/>
-        <origin rpy="0 0 0"
-                xyz="0 0 0"/>
-        <parent link="virtualLink_world"/>
-        <child link="virtualLink_body_front"/>
-    </joint>
-    <link name="virtualLink_body_front">
-        <origin rpy="0 0 0" xyz="0 0 0"/>
-    </link>
-    <joint name="joint_body_front_roll" type="continuous">
-        <axis xyz="1 0 0"/>
-        <origin rpy="0 0 0"
-                xyz="0 0 0"/>
-        <parent link="virtualLink_body_front"/>
-        <child link="body_front"/>
-    </joint>
-    <link name="body_front">
-        <visual>
-            <origin rpy="0 0 0"
-                    xyz="0 0 0"/>
-            <geometry>
-                <mesh filename="${robotPackagePath}/${modelDataResourseFolder}/body_front.dae"/>
-            </geometry>
-        </visual>
-    </link>
-    <joint name="joint_body_back_pitch" type="revolute">
-        <axis xyz="0 1 0"/>
-        <limit lower="${DEG2RAD*bodyPitchAngle_min}" effort="1000.0"
-               upper="${DEG2RAD*bodyPitchAngle_max}" velocity="0.5"/>
-        <origin rpy="0 0 0"
-                xyz="${-bodyFront_depth/2.0} 0 ${-bodyFront_height/2.0}"/>
-        <parent link="body_front"/>
-        <child link="body_link"/>
-    </joint>
-    <link name="body_link">
-        <visual>
-            <origin rpy="0 0 0"
-                    xyz="${-bodyLink_length/2.0} 0 ${bodyFront_height/2.0}"/>
-            <geometry>
-                <mesh filename="${robotPackagePath}/${modelDataResourseFolder}/body_link.dae"/>
-            </geometry>
-        </visual>
-    </link>
-    <joint name="joint_body_back_roll" type="continuous">
-        <axis xyz="1 0 0"/>
-        <origin rpy="0 0 0"
-                xyz="0 0 0"/>
-        <parent link="body_link"/>
-        <child link="body_back"/>
-    </joint>
-    <link name="body_back">
-        <visual>
-            <origin rpy="0 0 0"
-                    xyz="${-bodyLink_length - bodyBack_depth/2.0} 0 ${bodyBack_height/2.0}"/>
-            <geometry>
-                <mesh filename="${robotPackagePath}/${modelDataResourseFolder}/body_back.dae"/>
-            </geometry>
-        </visual>
-    </link>
-    <!-- FLIPPERS -->
-    <xacro:combine_lr_flippers
-            left_joint_name="joint_flipper_left" right_joint_name="joint_flipper_right"
-            parent="body_front" flipper_tread="${flipper_tread}" suffix="front">
-        <origin rpy="0 0 0" xyz="${flipperAxis_fromBodyCenter} 0 0"/>
-    </xacro:combine_lr_flippers>
-    <!-- WHEELS -->
-    <xacro:combine_lr_wheels
-            joint_name="joint_starwheel_front" parent="body_front"
-            suffix="front" wheel_tread="${frontwheel_tread}">
-        <origin rpy="0 0 0"
-                xyz="${frontwheelAxis_fromBodyCenter} 0 0"/>
-    </xacro:combine_lr_wheels>
-    <xacro:combine_lr_wheels
-            joint_name="joint_starwheel_back" parent="body_back"
-            suffix="back" wheel_tread="${backwheel_tread}">
-        <origin rpy="0 0 0"
-                xyz="${backwheelAxis_fromBodyCenter} 0 ${bodyBack_height/2.0}"/>
-    </xacro:combine_lr_wheels>
-    <!-- ARM BASE -->
+    <xacro:yozakura_body parent_link="root"/>
+    <!-- ARM -->
     <joint name="virtualjoint_arm_base" type="fixed">
         <origin rpy="0 0 0" xyz="${-armBase_fromBodyCenter_X} 0 ${bodyFront_height/2.0}"/>
@@ -99,78 +19,4 @@
         <origin rpy="0 0 0" xyz="0 0 0"/>
     </link>
-    <joint name="joint_arm_yaw" type="revolute">
-        <axis xyz="0 0 1"/>
-        <limit lower="${DEG2RAD*armYawAngle_min}" effort="1000.0"
-               upper="${DEG2RAD*armYawAngle_max}" velocity="0.5"/>
-        <origin rpy="0 0 0"
-                xyz="0 0 ${armYawStage_fromBodyTop}"/>
-        <parent link="virtual_arm_base"/>
-        <child link="arm_yaw"/>
-    </joint>
-    <link name="arm_yaw">
-        <visual>
-            <origin rpy="0 0 0"
-                    xyz="0 0 0"/>
-            <geometry>
-                <mesh filename="${robotPackagePath}/${modelDataResourseFolder}/arm_yaw.dae"/>
-            </geometry>
-        </visual>
-    </link>
-    <joint name="joint_arm_pitch" type="revolute">
-        <axis xyz="0 1 0"/>
-        <limit lower="${DEG2RAD*armPitchAngle_min}" effort="1000.0"
-               upper="${DEG2RAD*armPitchAngle_max}" velocity="0.5"/>
-        <origin rpy="0 0 0"
-                xyz="${-armPitchAxis_fromYawAxis} 0 ${armPitchAxis_fromYawStage}"/>
-        <parent link="arm_yaw"/>
-        <child link="arm_pitch"/>
-    </joint>
-    <link name="arm_pitch">
-        <visual>
-            <origin rpy="0 0 0"
-                    xyz="${-armLinearAxis_fromPitchAxis} 0	${-armPitchAxis_fromYawStage + armLinearAxis_fromYawStage}"/>
-            <geometry>
-                <mesh filename="${robotPackagePath}/${modelDataResourseFolder}/arm_pitch.dae"/>
-            </geometry>
-        </visual>
-    </link>
-    <!-- ARM BELLOWS -->
-    <joint name="virtualjoint_arm_bellows_base" type="fixed">
-        <origin rpy="0 0 0" xyz="0 0 ${-armLinearBase_ArmLinearAxis}"/>
-        <parent link="arm_pitch"/>
-        <child link="arm_linear_frame_base"/>
-    </joint>
-    <link name="arm_linear_frame_base">
-        <origin rpy="0 0 0" xyz="0 0 0"/>
-    </link>
-    <!-- right -->
-    <joint name="virtualJoint_armLinear_base_right" type="prismatic">
-        <axis xyz="0 1 0"/>
-        <limit lower="${DEG2RAD*armYawAngle_min}" effort="1000.0"
-               upper="${DEG2RAD*armYawAngle_max}" velocity="0.5"/>
-        <origin rpy="0 0 0" xyz="0 ${-armLinear_frame_length/2.0} 0"/>
-        <parent link="arm_linear_frame_base"/>
-        <child link="virtualLink_armLinear_base_right"/>
-    </joint>
-    <link name="virtualLink_armLinear_base_right">
-        <origin rpy="0 0 0" xyz="0 0 0"/>
-    </link>
-    <xacro:armjack_right parent="virtualLink_armLinear_base_right" suffix="1"/>
-    <xacro:armjack_right parent="${arm_linear_frame_right_B}_1" suffix="2"/>
-    <xacro:armjack_right parent="${arm_linear_frame_right_B}_2" suffix="3"/>
-    <!-- left -->
-    <joint name="virtualJoint_armLinear_base_left" type="prismatic">
-        <axis xyz="0 1 0"/>
-        <limit lower="${DEG2RAD*armYawAngle_min}" effort="1000.0"
-               upper="${DEG2RAD*armYawAngle_max}" velocity="0.5"/>
-        <origin rpy="0 0 0" xyz="0 ${armLinear_frame_length/2.0} 0"/>
-        <parent link="arm_linear_frame_base"/>
-        <child link="virtualLink_armLinear_base_left"/>
-    </joint>
-    <link name="virtualLink_armLinear_base_left">
-        <origin rpy="0 0 0" xyz="0 0 0"/>
-    </link>
-    <xacro:armjack_left parent="virtualLink_armLinear_base_left" suffix="1"/>
-    <xacro:armjack_left parent="${arm_linear_frame_left_B}_1" suffix="2"/>
-    <xacro:armjack_left parent="${arm_linear_frame_left_B}_2" suffix="3"/>
+    <xacro:yozakura_arm parent_link="virtual_arm_base"/>
 </robot>
