Commit message: add parameter for shifting the pos of urg

File: yozakura_display/robot/config.xacro (robot description, xacro)
@@ -3,4 +3,6 @@
     <property name="robotPackagePath" value="package://yozakura_display/robot"/>
     <property name="modelDataResourseFolder" value="daes"/>
+    <property name="urg_base_x" value="0.015"/>
+    <property name="urg_base_y" value="0.015"/>
     <property name="bodyFront_depth" value="0.262"/>
     <property name="bodyFront_height" value="0.072"/>
@@ -42,13 +44,3 @@
     <property name="armLinearBase_ArmLinearAxis" value="0.025"/>
     <property name="armLinear_frame_length" value="0.200"/>
-    <property name="arm_linear_frame_left_A" value="arm_linear_frame_left_A"/>
-    <property name="arm_linear_frame_left_B" value="arm_linear_frame_left_B"/>
-    <property name="joint_armLinear_left_A" value="joint_armLinear_left_A"/>
-    <property name="joint_armLinear_left_B" value="joint_armLinear_left_B"/>
-    <property name="joint_armLinear_left_C" value="joint_armLinear_left_C"/>
-    <property name="arm_linear_frame_right_A" value="arm_linear_frame_right_A"/>
-    <property name="arm_linear_frame_right_B" value="arm_linear_frame_right_B"/>
-    <property name="joint_armLinear_right_A" value="joint_armLinear_right_A"/>
-    <property name="joint_armLinear_right_B" value="joint_armLinear_right_B"/>
-    <property name="joint_armLinear_right_C" value="joint_armLinear_right_C"/>
 </robot>

File: yozakura_display/robot/define.xacro (robot description, xacro)
@@ -4,3 +4,13 @@
 	<property name="DEG2RAD" 	value= "0.017453293" />
 	<property name="RAD2DEG" 	value="57.295779513" />
+    <property name="arm_linear_frame_left_A" value="arm_linear_frame_left_A"/>
+    <property name="arm_linear_frame_left_B" value="arm_linear_frame_left_B"/>
+    <property name="joint_armLinear_left_A" value="joint_armLinear_left_A"/>
+    <property name="joint_armLinear_left_B" value="joint_armLinear_left_B"/>
+    <property name="joint_armLinear_left_C" value="joint_armLinear_left_C"/>
+    <property name="arm_linear_frame_right_A" value="arm_linear_frame_right_A"/>
+    <property name="arm_linear_frame_right_B" value="arm_linear_frame_right_B"/>
+    <property name="joint_armLinear_right_A" value="joint_armLinear_right_A"/>
+    <property name="joint_armLinear_right_B" value="joint_armLinear_right_B"/>
+    <property name="joint_armLinear_right_C" value="joint_armLinear_right_C"/>
 </robot>

File: yozakura_display/robot/yozakura.urdf.xacro (robot description, xacro)
@@ -10,4 +10,14 @@
     </link>
     <xacro:yozakura_body parent_link="root"/>
+    <!--URG-->
+    <joint name="virtualjoint_urg" type="fixed">
+        <origin rpy="0 0 0" xyz="0 0 0"/>
+        <parent link="body_front"/>
+        <child link="urg_base"/>
+    </joint>
+    <link name="urg_base">
+        <origin rpy="0 0 0"
+                xyz="${urg_base_x} ${urg_base_y} 0"/>
+    </link>
     <!-- ARM -->
     <joint name="virtualjoint_arm_base" type="fixed">

Commit message: arange the pos of urg

File: yozakura_display/robot/config.xacro (robot description, xacro)
@@ -3,6 +3,6 @@
     <property name="robotPackagePath" value="package://yozakura_display/robot"/>
     <property name="modelDataResourseFolder" value="daes"/>
-    <property name="urg_base_x" value="0.015"/>
-    <property name="urg_base_y" value="0.015"/>
+    <property name="urg_base_x" value="0.100"/>
+    <property name="urg_base_y" value="-0.050"/>
     <property name="bodyFront_depth" value="0.262"/>
     <property name="bodyFront_height" value="0.072"/>

File: yozakura_display/robot/yozakura.urdf.xacro (robot description, xacro)
@@ -12,11 +12,11 @@
     <!--URG-->
     <joint name="virtualjoint_urg" type="fixed">
-        <origin rpy="0 0 0" xyz="0 0 0"/>
+        <origin rpy="0 0 0"
+                xyz="${urg_base_x} ${urg_base_y} 0"/>
         <parent link="body_front"/>
         <child link="urg_base"/>
     </joint>
     <link name="urg_base">
-        <origin rpy="0 0 0"
-                xyz="${urg_base_x} ${urg_base_y} 0"/>
+        <origin rpy="0 0 0" xyz="0 0 0"/>
     </link>
     <!-- ARM -->

Commit message: 3DCG model

File: yozakura_display/robot/config.xacro (robot description, xacro)
@@ -3,7 +3,7 @@
     <property name="robotPackagePath" value="package://yozakura_display/robot"/>
     <property name="modelDataResourseFolder" value="daes"/>
-    <property name="urg_base_x" value="0.100"/>
-    <property name="urg_base_y" value="-0.050"/>
-    <property name="bodyFront_depth" value="0.262"/>
+    <property name="urg_base_x" value="0.150"/>
+    <property name="urg_base_y" value="0.0"/>
+    <property name="bodyFront_depth" value="0.312"/>
     <property name="bodyFront_height" value="0.072"/>
     <property name="bodyFront_width" value="0.262"/>
@@ -17,7 +17,7 @@
     <property name="starWheel_radius" value="0.134"/>
     <property name="starWheelAxis_radius" value="0.134"/>
-    <property name="frontwheelAxis_fromBodyCenter" value="0.070"/>
+    <property name="frontwheelAxis_fromBodyCenter" value="0.10"/>
     <property name="backwheelAxis_fromBodyCenter" value="-0.100"/>
-    <property name="frontwheel_tread" value="0.372"/>
+    <property name="frontwheel_tread" value="0.300"/>
     <!-- from outside to outside -->
     <property name="backwheel_tread" value="0.386"/>
@@ -36,6 +36,6 @@
     <property name="armPitchAngle_max" value="90"/>
     <property name="armPitchAngle_min" value="-90"/>
-    <property name="armBase_fromBodyCenter_X" value="0.040"/>
-    <property name="armYawStage_fromBodyTop" value="0.020"/>
+    <property name="armBase_fromBodyCenter_X" value="-0.061"/>
+    <property name="armYawStage_fromBodyTop" value="0.014"/>
     <property name="armPitchAxis_fromYawAxis" value="0.045"/>
     <property name="armPitchAxis_fromYawStage" value="0.045"/>

File: yozakura_display/robot/yozakura.urdf.xacro (robot description, xacro)
@@ -3,5 +3,5 @@
     <xacro:include filename="$(find yozakura_display)/robot/define.xacro"/>
     <xacro:include filename="$(find yozakura_display)/robot/config.xacro"/>
-    <xacro:include filename="$(find yozakura_display)/robot/yozakura_arm.urdf.xacro"/>
+    <xacro:include filename="$(find yozakura_display)/robot/yozakura_arm2016.urdf.xacro"/>
     <xacro:include filename="$(find yozakura_display)/robot/yozakura_body.urdf.xacro"/>
     <!-- BODY -->
@@ -10,14 +10,4 @@
     </link>
     <xacro:yozakura_body parent_link="root"/>
-    <!--URG-->
-    <joint name="virtualjoint_urg" type="fixed">
-        <origin rpy="0 0 0"
-                xyz="${urg_base_x} ${urg_base_y} 0"/>
-        <parent link="body_front"/>
-        <child link="urg_base"/>
-    </joint>
-    <link name="urg_base">
-        <origin rpy="0 0 0" xyz="0 0 0"/>
-    </link>
     <!-- ARM -->
     <joint name="virtualjoint_arm_base" type="fixed">

File: yozakura_display/robot/yozakura_body.urdf.xacro (robot description, xacro)
@@ -3,5 +3,4 @@
     <xacro:include filename="$(find yozakura_display)/robot/define.xacro"/>
     <xacro:include filename="$(find yozakura_display)/robot/config.xacro"/>
-    <xacro:include filename="$(find yozakura_display)/robot/flipper_macro.xacro"/>
     <xacro:include filename="$(find yozakura_display)/robot/wheel_macro.xacro"/>
     <xacro:macro name="yozakura_body" params="parent_link">
@@ -24,5 +23,5 @@
                 <origin rpy="0 0 0" xyz="0 0 0"/>
                 <geometry>
-                    <mesh filename="${robotPackagePath}/${modelDataResourseFolder}/body_front.dae"/>
+                    <mesh filename="${robotPackagePath}/${modelDataResourseFolder}/front_body.dae"/>
                 </geometry>
             </visual>
@@ -61,10 +60,4 @@
             </visual>
         </link>
-        <!-- FLIPPERS -->
-        <xacro:combine_lr_flippers
-                left_joint_name="joint_flipper_left" right_joint_name="joint_flipper_right"
-                parent="body_front" flipper_tread="${flipper_tread}" suffix="front">
-            <origin rpy="0 0 0" xyz="${flipperAxis_fromBodyCenter} 0 0"/>
-        </xacro:combine_lr_flippers>
         <!-- WHEELS -->
         <xacro:combine_lr_wheels
