Commit message: fit jointstate_publisher to new msg

File: yozakura_display/robot/yozakura.urdf.xacro (robot description, xacro)
@@ -37,5 +37,5 @@
         </visual>
     </link>
-    <joint name="joint_body_pitch" type="revolute">
+    <joint name="joint_body_back_pitch" type="revolute">
         <axis xyz="0 1 0"/>
         <limit lower="${DEG2RAD*bodyPitchAngle_min}" effort="1000.0"
@@ -55,5 +55,5 @@
         </visual>
     </link>
-    <joint name="joint_body_roll" type="continuous">
+    <joint name="joint_body_back_roll" type="continuous">
         <axis xyz="1 0 0"/>
         <origin rpy="0 0 0"

File: yozakura_display/robot/yozakura_body.urdf.xacro (robot description, xacro)
@@ -1,72 +1,72 @@
 <?xml version="1.0"?>
 <robot name="yozakura" xmlns:xacro="http://www.ros.org/wiki/xacro">
-	<xacro:include filename="$(find xacro)/define.xacro" />
-	<xacro:include filename="$(find yozakura_display)/robot/config.xacro" />
-	<xacro:include filename="$(find yozakura_display)/robot/flipper_macro.xacro" />
-	<xacro:include filename="$(find yozakura_display)/robot/starWheel_macro.xacro" />
-	<xacro:include filename="$(find yozakura_display)/robot/armjack_left_macro.xacro" />
-	<xacro:include filename="$(find yozakura_display)/robot/armjack_right_macro.xacro" />
-	<!-- BODY -->
-	<link name="body_front">
-		<visual>
-			<origin rpy="0 0 0"
-							xyz="0 0 0"/>
-			<geometry>
-				<mesh filename="${robotPackagePath}/${modelDataResourseFolder}/body_front.stl"/>
-			</geometry>
-		</visual>
-	</link>
-  <joint name="joint_body_pitch" type="revolute">
-    <axis xyz="0 1 0"/>
-    <limit 	lower="${DEG2RAD*bodyPitchAngle_min}" effort="1000.0"
-						upper="${DEG2RAD*bodyPitchAngle_max}" velocity="0.5"/>
-    <origin rpy="0 0 0"
-						xyz="${-bodyFront_depth/2.0} 0 ${-bodyFront_height/2.0}"/>
-    <parent link="body_front"/>
-    <child link="body_link"/>
-  </joint>
-	<link name="body_link">
-		<visual>
-			<origin rpy="0 0 0"
-							xyz="${-bodyLink_length/2.0} 0 ${bodyFront_height/2.0}"/>
-			<geometry>
-				<mesh filename="${robotPackagePath}/${modelDataResourseFolder}/body_link.stl"/>
-			</geometry>
-		</visual>
-	</link>
-  <joint name="joint_body_roll" type="continuous">
-    <axis xyz="1 0 0"/>
-    <origin rpy="0 0 0"
-						xyz="0 0 0"/>
-    <parent link="body_link"/>
-    <child link="body_back"/>
-  </joint>
-	<link name="body_back">
-		<visual>
-			<origin rpy="0 0 0"
-							xyz="${-bodyLink_length - bodyBack_depth/2.0} 0 ${bodyBack_height/2.0}"/>
-			<geometry>
-				<mesh filename="${robotPackagePath}/${modelDataResourseFolder}/body_back.stl"/>
-			</geometry>
-		</visual>
-	</link>
-	<!-- FLIPPERS -->
-	<xacro:combine_lr_flippers
-									left_joint_name="joint_flipper_left" right_joint_name="joint_flipper_right"
-									parent="body_front" flipper_tread="${flipper_tread}" suffix="front">
-		<origin rpy="0 0 0" xyz="${flipperAxis_fromBodyCenter} 0 0"/>
-	</xacro:combine_lr_flippers>
-	<!-- WHEELS -->
-	<xacro:combine_lr_wheels
-									joint_name="joint_starwheel_front" parent="body_front"
-									suffix="front" wheel_tread="${frontwheel_tread}">
-		<origin rpy="0 0 0"
-						xyz="${frontwheelAxis_fromBodyCenter} 0 0" />
-	</xacro:combine_lr_wheels>
-	<xacro:combine_lr_wheels
-									joint_name="joint_starwheel_back" parent="body_back"
-									suffix="back" wheel_tread="${backwheel_tread}">
-		<origin rpy="0 0 0"
-						xyz="${backwheelAxis_fromBodyCenter} 0 ${bodyBack_height/2.0}" />
-	</xacro:combine_lr_wheels>
+    <xacro:include filename="$(find xacro)/define.xacro"/>
+    <xacro:include filename="$(find yozakura_display)/robot/config.xacro"/>
+    <xacro:include filename="$(find yozakura_display)/robot/flipper_macro.xacro"/>
+    <xacro:include filename="$(find yozakura_display)/robot/starWheel_macro.xacro"/>
+    <xacro:include filename="$(find yozakura_display)/robot/armjack_left_macro.xacro"/>
+    <xacro:include filename="$(find yozakura_display)/robot/armjack_right_macro.xacro"/>
+    <!-- BODY -->
+    <link name="body_front">
+        <visual>
+            <origin rpy="0 0 0"
+                    xyz="0 0 0"/>
+            <geometry>
+                <mesh filename="${robotPackagePath}/${modelDataResourseFolder}/body_front.stl"/>
+            </geometry>
+        </visual>
+    </link>
+    <joint name="joint_body_pitch" type="revolute">
+        <axis xyz="0 1 0"/>
+        <limit lower="${DEG2RAD*bodyPitchAngle_min}" effort="1000.0"
+               upper="${DEG2RAD*bodyPitchAngle_max}" velocity="0.5"/>
+        <origin rpy="0 0 0"
+                xyz="${-bodyFront_depth/2.0} 0 ${-bodyFront_height/2.0}"/>
+        <parent link="body_front"/>
+        <child link="body_link"/>
+    </joint>
+    <link name="body_link">
+        <visual>
+            <origin rpy="0 0 0"
+                    xyz="${-bodyLink_length/2.0} 0 ${bodyFront_height/2.0}"/>
+            <geometry>
+                <mesh filename="${robotPackagePath}/${modelDataResourseFolder}/body_link.stl"/>
+            </geometry>
+        </visual>
+    </link>
+    <joint name="joint_body_roll" type="continuous">
+        <axis xyz="1 0 0"/>
+        <origin rpy="0 0 0"
+                xyz="0 0 0"/>
+        <parent link="body_link"/>
+        <child link="body_back"/>
+    </joint>
+    <link name="body_back">
+        <visual>
+            <origin rpy="0 0 0"
+                    xyz="${-bodyLink_length - bodyBack_depth/2.0} 0 ${bodyBack_height/2.0}"/>
+            <geometry>
+                <mesh filename="${robotPackagePath}/${modelDataResourseFolder}/body_back.stl"/>
+            </geometry>
+        </visual>
+    </link>
+    <!-- FLIPPERS -->
+    <xacro:combine_lr_flippers
+            left_joint_name="joint_flipper_left" right_joint_name="joint_flipper_right"
+            parent="body_front" flipper_tread="${flipper_tread}" suffix="front">
+        <origin rpy="0 0 0" xyz="${flipperAxis_fromBodyCenter} 0 0"/>
+    </xacro:combine_lr_flippers>
+    <!-- WHEELS -->
+    <xacro:combine_lr_wheels
+            joint_name="joint_starwheel_front" parent="body_front"
+            suffix="front" wheel_tread="${frontwheel_tread}">
+        <origin rpy="0 0 0"
+                xyz="${frontwheelAxis_fromBodyCenter} 0 0"/>
+    </xacro:combine_lr_wheels>
+    <xacro:combine_lr_wheels
+            joint_name="joint_starwheel_back" parent="body_back"
+            suffix="back" wheel_tread="${backwheel_tread}">
+        <origin rpy="0 0 0"
+                xyz="${backwheelAxis_fromBodyCenter} 0 ${bodyBack_height/2.0}"/>
+    </xacro:combine_lr_wheels>
 </robot>

Commit message: 3DCG_with urg

File: yozakura_display/robot/yozakura.urdf.xacro (robot description, xacro)
@@ -9,5 +9,13 @@
         <origin rpy="0 0 0" xyz="0 0 0"/>
     </link>
-    <xacro:yozakura_body parent_link="root"/>
+   <joint name="root_center" type="fixed">
+          <origin rpy="0 0 0"  xyz="0 0 0.1"/>
+          <parent link="root"/>
+          <child link="center_yozakura"/>
+    </joint>
+    <link name="center_yozakura">
+         <origin rpy="0 0 0" xyz="0 0 0"/>
+    </link>
+    <xacro:yozakura_body parent_link="center_yozakura"/>
     <!-- ARM -->
     <joint name="virtualjoint_arm_base" type="fixed">
