Commit message: laser_scan

File: yozakura_display/robot/yozakura_arm2016.urdf.xacro (robot description, xacro)
@@ -29,7 +29,7 @@
                 xyz="0.060 0 0"/>
         <parent link="arm_yaw"/>
-        <child link="urg_base"/>
+        <child link="laser_link"/>
   </joint>
-  <link name="urg_base">
+  <link name="laser_link">
       <visual>
         <origin rpy="0 0 0" xyz="0 0 0.035"/>
